File: LNA-2W.kicad_pcb (KiCad board)
At the start: 2 copper layers, 58.2 x 30 mm, 30 parts, among them J1 SMA_Edge, J2 SMA_Edge, U1 TQP7M9106

Commit message: Add files via upload
Other:
- board text added: "RF-IN"
- board text added: "RF-OUT"
Changed lines of the file:
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@@
 			(at 5.5 -0.09685 90)
 			(layer "F.Fab")
+			(hide yes)
 			(effects
 				(font
@@
 			(at -5.5 0 90)
 			(layer "F.Fab")
+			(hide yes)
 			(effects
 				(font
@@
 		(layer "Edge.Cuts")
 	)
+	(gr_text "RF-IN"
+		(at 108.75 103.75 0)
+		(layer "F.SilkS")
+		(effects
+			(font
+				(size 1 1)
+				(thickness 0.25)
+				(bold yes)
+			)
+			(justify left bottom)
+		)
+	)
+	(gr_text "RF-OUT"
+		(at 159.25 104.25 0)
+		(layer "F.SilkS")
+		(effects
+			(font
+				(size 1 1)
+				(thickness 0.25)
+				(bold yes)
+			)
+			(justify left bottom)
+		)
+	)
 	(segment
 		(start 118.675 108.25)
@@
 		(polygon
 			(pts
-				(xy 108 90) (xy 166.5 90) (xy 166.5 90) (xy 166.5 107) (xy 108 107)
+				(xy 108 90) (xy 166.5 90) (xy 166.5 107) (xy 108 107)
 			)
 		)
