File: LNA-2W.kicad_sch (KiCad schematic)
At the start: 30 parts, among them J1 SMA_Edge, J2 SMA_Edge, U1 TQP7M9106

Commit message: Add files via upload
Parts:
- J1: value SMA_Edge -> SMA_RF IN
- J2: value SMA_Edge -> SMA_RF OUT
Changed lines of the file:
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@@
 			)
 		)
-		(property "Value" "SMA_Edge"
+		(property "Value" "SMA_RF OUT"
 			(at 210.82 119.6731 0)
 			(effects
@@
 			)
 		)
-		(property "Value" "SMA_Edge"
+		(property "Value" "SMA_RF IN"
 			(at 43.18 119.0867 0)
 			(effects

Commit message: Add files via upload
Parts:
- removed C2: 2p4, Capacitor_SMD:C_0603_1608Metric, symbol Device:C_Small
- removed D1: SM05T1G, Package_TO_SOT_SMD:SOT-23-3, symbol Device:D_Zener_Dual_CommonAnode_KKA
- removed L1: 8n2, Inductor_SMD:L_0603_1608Metric, symbol Device:L_Small
- removed R1: 0R, Resistor_SMD:R_0603_1608Metric, symbol Device:R_Small
- added C1: 100p, Capacitor_SMD:C_0603_1608Metric, symbol Device:C_Small
- added C3: 8p2, Capacitor_SMD:C_0603_1608Metric, symbol Device:C_Small
- added C7: 22p, Capacitor_SMD:C_0603_1608Metric, symbol Device:C_Small
- added L3: 4n7, Inductor_SMD:L_0603_1608Metric, symbol Device:L_Small
- added R2: 4R3, Resistor_SMD:R_0603_1608Metric, symbol Device:R_Small
- C10: renamed from C8; value 100p -> 1n
- C2: renamed from C1; value 22p -> 100p
- C4: renamed from C3; value 6p8 -> 15p
- C6: renamed from C5; value 100p -> 6p8
- C8: renamed from C6; value 100n -> 100p
- L2: renamed from L3; footprint Inductor_SMD:L_Coilcraft_0805HQ_2012Metric -> Inductor_SMD:L_1008_2520Metric
- R3: value 240R -> 280R
- renumbered C9 to C11, C10 to C12, C11 to C13, C4 to C5, C7 to C9, L2 to L1, R2 to R1
Connections:
- net GND: now also C6.1, C3.2
- net at C2.1, R1.1: now also C1.2
- net at C2.2, R1.2: now also C3.1, R2.1
- net at C5.1, L2.2, U1.14 (RF_OUT/VCC)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: now also L3.1; no longer C6.1
- net at C4.1, U1.4 (RF_IN), U1.5 (RF_IN): now also R2.2
- net at J1.1 (In): now also C1.1
- net at C6.2: now also C7.1, L3.2; no longer FL1.1 (IN)
- new net: C7.2, FL1.1 (IN)
Other:
- title: LNA 2W -> LNA 2W 
- moved on the sheet: C6, FL1, J2
